File: BMS_5S_v2/BMS_5S_v2.kicad_pcb (KiCad board)
At the start: 4 copper layers, 50 x 95 mm, 132 parts, among them IC1 L99BM114-TR, J3 Conector, J4 Conn_02x02_Counter_Clockwise, J5 Conn_02x02_Counter_Clockwise, Q1 STL8N10LF3, Q2 STD105N10F7AG, T1 HMU2103NL, T2 HMU2103NL, U2 USBLC6-2SC6, U3 USBLC6-2SC6

Commit message: fix(silkscreen): correct J5 label from DAISE OUT to DAISY OUT and update renders
Parts:
- removed kibuzzard-6AD804A2: G***, kibuzzard-6AD804A2
- removed kibuzzard-6AD804BC: G***, kibuzzard-6AD804BC
- added kibuzzard-6AD93452: G***, kibuzzard-6AD93452, F.Cu at (148.9, 48.8)
- added kibuzzard-6AD93460: G***, kibuzzard-6AD93460, F.Cu at (145.7, 55.9)

Commit message: fix: resolve hardware audit issues, update documentation, fabrication package, and 3D renders
Parts:
- added kibuzzard-6ADA909C: G***, kibuzzard-6ADA909C, F.Cu at (127.0, 87.4)
- added kibuzzard-6ADA9153: G***, kibuzzard-6ADA9153, F.Cu at (147.5, 66.6)
- added kibuzzard-6ADA916E: G***, kibuzzard-6ADA916E, F.Cu at (147.5, 76.5)
- Q2: value STD105N10F7AG -> Q_NMOS_GDS
- moved Q2 1.59 mm to (131.6, 122.3), turned to -90 degrees
- renumbered STATUS to D4
Connections:
- Q2 pad 1: AGND -> Net-(Q2-G)
- Q2 pad 2: Net-(Q2-G) -> AGND
Routing:
- net GND_ESD: track 116.3 -> 127.6 mm
- net AGND: track 28.4 -> 34.7 mm, vias 27 -> 30
- net Net-(Q2-G): track 12.9 -> 11.7 mm
Other:
- board text added: "- 6.5 mm - GALVANIC ISOLATION BARRIER"
- board text removed: "- 10mm - GALVANIC ISOLATION BARRIER"
- board text removed: "HV ACCUMULATOR DOMAIN"
- board text removed: "ISOLATED LV DOMAIN"
