File: BMS_5S_v2/Power_Management.kicad_sch (KiCad schematic)
At the start: 18 parts, among them Q1 STL8N10LF3, Q2 STD105N10F7AG

Commit message: fix: resolve hardware audit issues, update documentation, fabrication package, and 3D renders
Parts:
- removed Q2: STD105N10F7AG, Package_TO_SOT_SMD:TO-252-2, symbol Transistor_FET:Q_NMOS_DGS
- added Q2: Q_NMOS_GDS, Package_TO_SOT_SMD:TO-252-2, symbol Transistor_FET:Q_NMOS_GDS
Connections:
- net AGND: now also Q2.2 (D)
- net GND_ESD: now also Q2.3 (S)
- net at C6.2, R2.2: now also Q2.1 (G)
Other:
- moved on the sheet: R3
Changed lines of the file:
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@@
 	(wire
 		(pts
-			(xy 205.74 105.41) (xy 214.63 105.41)
+			(xy 205.74 110.49) (xy 214.63 110.49)
 		)
 		(stroke
@@
 	(wire
 		(pts
-			(xy 191.77 105.41) (xy 191.77 96.52)
+			(xy 191.77 110.49) (xy 191.77 96.52)
 		)
 		(stroke
@@
 	(wire
 		(pts
-			(xy 200.66 105.41) (xy 191.77 105.41)
+			(xy 200.66 110.49) (xy 191.77 110.49)
 		)
 		(stroke
@@
 	(wire
 		(pts
-			(xy 214.63 105.41) (xy 214.63 96.52)
+			(xy 214.63 110.49) (xy 214.63 96.52)
 		)
 		(stroke
@@
 	)
 	(symbol
-		(lib_id "Transistor_FET:Q_NMOS_DGS")
-		(at 203.2 93.98 90)
-		(mirror x)
+		(lib_id "power:PWR_FLAG")
+		(at 181.61 96.52 0)
 		(unit 1)
 		(body_style 1)
@@
 		(in_pos_files yes)
 		(dnp no)
-		(property "Reference" "Q2"
-			(at 203.2 100.33 90)
+		(property "Reference" "#FLG05"
+			(at 181.61 98.425 0)
+			(hide yes)
 			(show_name no)
 			(do_not_autoplace no)
@@
 			)
 		)
-		(property "Value" "STD105N10F7AG"
-			(at 203.2 102.87 90)
+		(property "Value" "PWR_FLAG"
+			(at 181.61 92.71 0)
 			(hide yes)
 			(show_name no)
@@
 			)
 		)
-		(property "Footprint" "Package_TO_SOT_SMD:TO-252-2"
-			(at 200.66 99.06 0)
+		(property "Footprint" ""
+			(at 181.61 96.52 0)
 			(hide yes)
 			(show_name no)
@@
 		)
 		(property "Datasheet" ""
-			(at 203.2 93.98 0)
+			(at 181.61 96.52 0)
 			(hide yes)
 			(show_name no)
@@
 			)
 		)
-		(property "Description" "N-MOSFET transistor, drain/gate/source"
-			(at 203.2 93.98 0)
+		(property "Description" "Special symbol for telling ERC where power comes from"
+			(at 181.61 96.52 0)
 			(hide yes)
 			(show_name no)
@@
 			)
 		)
-		(pin "2"
-		)
-		(pin "3"
-		)
 		(pin "1"
 		)
@@
 			(project "BMS_5S_v2"
 				(path "/068efd84-10fe-4814-92cc-0cd9d996861a/4eab94bb-4cb7-463b-8254-02fb5fd547db"
-					(reference "Q2")
+					(reference "#FLG05")
 					(unit 1)
 				)
@@
 	)
 	(symbol
-		(lib_id "power:PWR_FLAG")
-		(at 181.61 96.52 0)
+		(lib_id "power:GND")
+		(at 175.26 46.99 0)
+		(mirror y)
 		(unit 1)
 		(body_style 1)
@@
 		(in_pos_files yes)
 		(dnp no)
-		(property "Reference" "#FLG05"
-			(at 181.61 98.425 0)
+		(property "Reference" "#PWR01"
+			(at 175.26 53.34 0)
 			(hide yes)
 			(show_name no)
@@
 			)
 		)
-		(property "Value" "PWR_FLAG"
-			(at 181.61 92.71 0)
-			(hide yes)
+		(property "Value" "AGND"
+			(at 175.26 51.054 0)
 			(show_name no)
 			(do_not_autoplace no)
@@
 		)
 		(property "Footprint" ""
-			(at 181.61 96.52 0)
+			(at 175.26 46.99 0)
 			(hide yes)
 			(show_name no)
@@
 		)
 		(property "Datasheet" ""
-			(at 181.61 96.52 0)
+			(at 175.26 46.99 0)
 			(hide yes)
 			(show_name no)
@@
 			)
 		)
-		(property "Description" "Special symbol for telling ERC where power comes from"
-			(at 181.61 96.52 0)
+		(property "Description" "Power symbol creates a global label with name \"GND\" , ground"
+			(at 175.26 46.99 0)
 			(hide yes)
 			(show_name no)
@@
 			(project "BMS_5S_v2"
 				(path "/068efd84-10fe-4814-92cc-0cd9d996861a/4eab94bb-4cb7-463b-8254-02fb5fd547db"
-					(reference "#FLG05")
+					(reference "#PWR01")
 					(unit 1)
 				)
@@
 	)
 	(symbol
-		(lib_id "power:GND")
-		(at 175.26 46.99 0)
-		(mirror y)
+		(lib_id "power:VCC")
+		(at 100.33 83.82 0)
 		(unit 1)
 		(body_style 1)
@@
 		(in_pos_files yes)
 		(dnp no)
-		(property "Reference" "#PWR01"
-			(at 175.26 53.34 0)
+		(property "Reference" "#PWR010"
+			(at 100.33 87.63 0)
 			(hide yes)
 			(show_name no)
@@
 			)
 		)
-		(property "Value" "AGND"
-			(at 175.26 51.054 0)
+		(property "Value" "VTREF"
+			(at 100.33 80.01 0)
 			(show_name no)
 			(do_not_autoplace no)
@@
 		)
 		(property "Footprint" ""
-			(at 175.26 46.99 0)
+			(at 100.33 83.82 0)
 			(hide yes)
 			(show_name no)
@@
 		)
 		(property "Datasheet" ""
-			(at 175.26 46.99 0)
+			(at 100.33 83.82 0)
 			(hide yes)
 			(show_name no)
@@
 			)
 		)
-		(property "Description" "Power symbol creates a global label with name \"GND\" , ground"
-			(at 175.26 46.99 0)
+		(property "Description" "Power symbol creates a global label with name \"VCC\""
+			(at 100.33 83.82 0)
 			(hide yes)
 			(show_name no)
@@
 			(project "BMS_5S_v2"
 				(path "/068efd84-10fe-4814-92cc-0cd9d996861a/4eab94bb-4cb7-463b-8254-02fb5fd547db"
-					(reference "#PWR01")
+					(reference "#PWR010")
 					(unit 1)
 				)
@@
 	)
 	(symbol
-		(lib_id "power:VCC")
-		(at 100.33 83.82 0)
+		(lib_id "Device:C_Small")
+		(at 96.52 91.44 0)
 		(unit 1)
 		(body_style 1)
@@
 		(in_pos_files yes)
 		(dnp no)
-		(property "Reference" "#PWR010"
-			(at 100.33 87.63 0)
-			(hide yes)
+		(property "Reference" "C9"
+			(at 98.806 90.424 0)
 			(show_name no)
 			(do_not_autoplace no)
@@
 					(size 1.27 1.27)
 				)
+				(justify left)
 			)
 		)
-		(property "Value" "VTREF"
-			(at 100.33 80.01 0)
+		(property "Value" "2u2F/16V"
+			(at 98.806 92.456 0)
 			(show_name no)
 			(do_not_autoplace no)
@@
 					(size 1.27 1.27)
 				)
+				(justify left)
 			)
 		)
-		(property "Footprint" ""
-			(at 100.33 83.82 0)
+		(property "Footprint" "Capacitor_SMD:C_0805_2012Metric_Pad1.18x1.45mm_HandSolder"
+			(at 96.52 91.44 0)
 			(hide yes)
 			(show_name no)
@@
 		)
 		(property "Datasheet" ""
-			(at 100.33 83.82 0)
+			(at 96.52 91.44 0)
 			(hide yes)
 			(show_name no)
@@
 			)
 		)
-		(property "Description" "Power symbol creates a global label with name \"VCC\""
-			(at 100.33 83.82 0)
+		(property "Description" "Unpolarized capacitor, small symbol"
+			(at 96.52 91.44 0)
 			(hide yes)
 			(show_name no)
@@
 			)
 		)
+		(pin "2"
+		)
 		(pin "1"
 		)
@@
 			(project "BMS_5S_v2"
 				(path "/068efd84-10fe-4814-92cc-0cd9d996861a/4eab94bb-4cb7-463b-8254-02fb5fd547db"
-					(reference "#PWR010")
+					(reference "C9")
 					(unit 1)
 				)
@@
 	)
 	(symbol
-		(lib_id "Device:C_Small")
-		(at 96.52 91.44 0)
+		(lib_id "Transistor_FET:Q_NMOS_GDS")
+		(at 203.2 93.98 90)
+		(mirror x)
 		(unit 1)
 		(body_style 1)
@@
 		(in_pos_files yes)
 		(dnp no)
-		(property "Reference" "C9"
-			(at 98.806 90.424 0)
+		(property "Reference" "Q2"
+			(at 203.2 100.33 90)
 			(show_name no)
 			(do_not_autoplace no)
@@
 					(size 1.27 1.27)
 				)
-				(justify left)
 			)
 		)
-		(property "Value" "2u2F/16V"
-			(at 98.806 92.456 0)
+		(property "Value" "Q_NMOS_GDS"
+			(at 203.2 102.87 90)
 			(show_name no)
 			(do_not_autoplace no)
@@
 					(size 1.27 1.27)
 				)
-				(justify left)
 			)
 		)
-		(property "Footprint" "Capacitor_SMD:C_0805_2012Metric_Pad1.18x1.45mm_HandSolder"
-			(at 96.52 91.44 0)
+		(property "Footprint" "Package_TO_SOT_SMD:TO-252-2"
+			(at 200.66 99.06 0)
 			(hide yes)
 			(show_name no)
@@
 		)
 		(property "Datasheet" ""
-			(at 96.52 91.44 0)
+			(at 203.2 93.98 0)
 			(hide yes)
 			(show_name no)
@@
 			)
 		)
-		(property "Description" "Unpolarized capacitor, small symbol"
-			(at 96.52 91.44 0)
+		(property "Description" "N-MOSFET transistor, gate/drain/source"
+			(at 203.2 93.98 0)
 			(hide yes)
 			(show_name no)
@@
 			)
 		)
+		(pin "1"
+		)
 		(pin "2"
 		)
-		(pin "1"
+		(pin "3"
 		)
 		(instances
 			(project "BMS_5S_v2"
 				(path "/068efd84-10fe-4814-92cc-0cd9d996861a/4eab94bb-4cb7-463b-8254-02fb5fd547db"
-					(reference "C9")
+					(reference "Q2")
 					(unit 1)
 				)
@@
 	(symbol
 		(lib_id "Device:R_Small")
-		(at 203.2 105.41 90)
+		(at 203.2 110.49 90)
 		(mirror x)
 		(unit 1)
@@
 		(dnp no)
 		(property "Reference" "R3"
-			(at 203.2 103.632 90)
+			(at 203.2 108.712 90)
 			(show_name no)
 			(do_not_autoplace no)
@@
 		)
 		(property "Value" "47"
-			(at 203.2 107.442 90)
+			(at 203.2 112.522 90)
 			(show_name no)
 			(do_not_autoplace no)
@@
 		)
 		(property "Footprint" "Resistor_SMD:R_2512_6332Metric_Pad1.40x3.35mm_HandSolder"
-			(at 203.2 105.41 0)
+			(at 203.2 110.49 0)
 			(hide yes)
 			(show_name no)
@@
 		)
 		(property "Datasheet" ""
-			(at 203.2 105.41 0)
+			(at 203.2 110.49 0)
 			(hide yes)
 			(show_name no)
@@
 		)
 		(property "Description" "Resistor, small symbol"
-			(at 203.2 105.41 0)
+			(at 203.2 110.49 0)
 			(hide yes)
 			(show_name no)
